File: Circuit(KiCad-ver.5)/DACAP/MD&SubCPU-ver2.0.sch (KiCad schematic (older format))
At the start: 85 parts, among them J1 Battery, J10 Raspberry_Pi_2_3, J11 Servo, J12 Motor-ONOFF, J13 Servo-ONOFF, J14 MPU9250, J15 PI-I2C, J16 Motor, J17 USB_B_Micro, J2 ST-I2C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

Commit message: upgrade circuit
Parts:
- removed C13: 220uF, Capacitor_SMD:CP_Elec_8x10, symbol Device:CP
- removed C14, C7: 10uF, Capacitor_SMD:C_0805_2012Metric_Pad1.15x1.40mm_HandSolder, symbol Device:CP1_Small
- removed C15, C8: tantalum 10uF, Capacitor_Tantalum_SMD:CP_EIA-3216-12_Kemet-S_Pad1.58x1.35mm_HandSolder, symbol Device:CP1_Small
- removed F3: Polyfuse, Resistor_THT:R_Axial_DIN0207_L6.3mm_D2.5mm_P10.16mm_Horizontal, symbol Device:Polyfuse
- removed J16: Motor, zisaku:Ultra_male, symbol Connector:Conn_01x02_Male
- removed J17: USB_B_Micro, zisaku:microusbB-supply, symbol Connector:USB_B_Micro
- removed J4: Encoder data, Connector_JST:JST_EH_S06B-EH_1x06_P2.50mm_Horizontal, symbol Connector:Conn_01x06_Female
- removed LS2: PKM13EPYH4000-A0, Buzzer_Beeper:Buzzer_TDK_PS1240P02BT_D12.2mm_H6.5mm, symbol Device:Speaker
- removed R14, R25: 121 1%, Resistor_SMD:R_0805_2012Metric_Pad1.15x1.40mm_HandSolder, symbol Device:R
- removed R16, R26: 365 1%, Resistor_SMD:R_0805_2012Metric_Pad1.15x1.40mm_HandSolder, symbol Device:R
- removed U3, U4: LM1085IS-5.0/NOPB, Package_TO_SOT_SMD:TO-263-3_TabPin2, symbol Regulator_Linear:LM1085-5.0
- added C7, C8: 1uF, Capacitor_SMD:C_0805_2012Metric_Pad1.15x1.40mm_HandSolder, symbol Device:C_Small
- added J4: Encoder, Connector_JST:JST_EH_S7B-EH_1x07_P2.50mm_Horizontal, symbol Connector:Conn_01x07_Female
- added M1: Motor_DC, zisaku:Ultra_female, symbol Motor:Motor_DC
- added U3: MCP1703A-3302_SOT23, Package_TO_SOT_SMD:SOT-23, symbol Regulator_Linear:MCP1703A-3302_SOT23
- J1: footprint zisaku:Ultra_female -> zisaku:Ultra_male
- J14: value MPU9250 -> MPU6050
- J6: value +5V -> Fun0
- J7: value +5V -> Fun1
- R10, R15, R20, R21, R23, R24: value 1k -> 100
- R18, R19: value 2.2k -> 680
- R2: value 4.7k -> 680
Connections:
- net +3V3: now also J14.1 (Pin_1), C8.1, J4.1 (Pin_1), J4.2 (Pin_2), U3.2 (VO); no longer J14.2 (Pin_2)
- net GND: now also J14.2 (Pin_2), C7.2, C8.2, J4.3 (Pin_3), U3.1 (GND); no longer J14.3 (Pin_3)
- net OUTA: now also M1.1 (+)
- net OUTB: now also M1.2 (-)
- net PI-SCL: now also J14.3 (Pin_3); no longer J14.4 (Pin_4)
- net PI-SDA: now also J14.4 (Pin_4); no longer J14.5 (Pin_5)
- net ST-SCL: now also J4.4 (Pin_4)
- net ST-SDA: now also J4.5 (Pin_5)
- net VCC: now also C7.1, U3.3 (VI)
- net buzz: now reaches LS1.1, U2.15 (PB1)
- net buzz: now also J10.37 (GPIO26)
- net Encoder0 renamed EncoderA
- net EncoderA: now also J4.6 (Pin_6)
- net Encoder1 renamed EncoderB
- net EncoderB: now also J4.7 (Pin_7)
- net Encoder2: no longer names the net of U2.13 (PA7)
- net Encoder3: no longer names the net of U2.18 (PA8)
- no-connect marks 8 -> 26
Other:
- moved on the sheet: C1, C10, C12, C2, C3, C4, C5, C6, C9, D1, D2, D3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
